File: h-bridge-inverter/h-bridge-inverter.kicad_sch (KiCad schematic)
At the start: 0 parts

Commit message: sine and triangular generation ok
Parts:
- added C1: 10u, symbol Device:C
- added Q1: PMOS, symbol Simulation_SPICE:PMOS
- added Q2: NPN, symbol Simulation_SPICE:NPN
- added R1, R3, R4: 10k, symbol Device:R
- added R2: 470, symbol Device:R
- added V1: 12, symbol Simulation_SPICE:VDC
- added V2: VPULSE, symbol Simulation_SPICE:VPULSE
Connections:
- new net: Q2.1 (C), R2.1
- new net: Q1.3 (S), R4.1, V1.1
- new net 0: C1.2, Q2.3 (E), R1.2, R3.2, V1.2, V2.2
- new net VOUT: C1.1, Q1.1 (D), R3.1
- new net VPULSE: Q2.2 (B), R1.1, V2.1
- new net VTRIG: Q1.2 (G), R2.2, R4.2
Other:
- added sheet Control (control.kicad_sch)
- note added: ".tran 10u 500m 10m"
